File: ClapDetectorPCB.kicad_pcb (KiCad board)
At the start: 2 copper layers, 0 parts

Commit message: Milestone 1
Parts:
- added BlueC: C_Rect_L7.0mm_W2.5mm_P5.00mm, Capacitor_THT:C_Rect_L7.0mm_W2.5mm_P5.00mm, F.Cu at (76.8, 203.0)
- added MIC: PinHeader_1x02_P2.54mm_Vertical, Connector_PinHeader_2.54mm:PinHeader_1x02_P2.54mm_Vertical, F.Cu at (47.5, 216.5)
- added OP-AMP: DIP-8_W7.62mm, Package_DIP:DIP-8_W7.62mm, F.Cu at (71.5, 214.0)
- added Potentiometer: Potentiometer_Vishay_T73YP_Vertical, Potentiometer_THT:Potentiometer_Vishay_T73YP_Vertical, F.Cu at (58.5, 234.0)
- added R: R_Axial_DIN0207_L6.3mm_D2.5mm_P7.62mm_Horizontal, Resistor_THT:R_Axial_DIN0207_L6.3mm_D2.5mm_P7.62mm_Horizontal, F.Cu at (67.5, 211.1)
- added R: R_Axial_DIN0207_L6.3mm_D2.5mm_P7.62mm_Horizontal, Resistor_THT:R_Axial_DIN0207_L6.3mm_D2.5mm_P7.62mm_Horizontal, F.Cu at (42.5, 222.8)
- added R: R_Axial_DIN0207_L6.3mm_D2.5mm_P7.62mm_Horizontal, Resistor_THT:R_Axial_DIN0207_L6.3mm_D2.5mm_P7.62mm_Horizontal, F.Cu at (83.0, 218.5)
- added R: R_Axial_DIN0207_L6.3mm_D2.5mm_P7.62mm_Horizontal, Resistor_THT:R_Axial_DIN0207_L6.3mm_D2.5mm_P7.62mm_Horizontal, F.Cu at (59.0, 203.5)
- added R: R_Axial_DIN0207_L6.3mm_D2.5mm_P7.62mm_Horizontal, Resistor_THT:R_Axial_DIN0207_L6.3mm_D2.5mm_P7.62mm_Horizontal, F.Cu at (79.2, 225.2)
- added R: R_Axial_DIN0207_L6.3mm_D2.5mm_P7.62mm_Horizontal, Resistor_THT:R_Axial_DIN0207_L6.3mm_D2.5mm_P7.62mm_Horizontal, F.Cu at (63.8, 218.1)
- added R: R_Axial_DIN0207_L6.3mm_D2.5mm_P7.62mm_Horizontal, Resistor_THT:R_Axial_DIN0207_L6.3mm_D2.5mm_P7.62mm_Horizontal, F.Cu at (47.5, 203.7)
- added R: R_Axial_DIN0207_L6.3mm_D2.5mm_P7.62mm_Horizontal, Resistor_THT:R_Axial_DIN0207_L6.3mm_D2.5mm_P7.62mm_Horizontal, F.Cu at (61.3, 220.1)
- added YellowC: C_Rect_L7.0mm_W2.5mm_P5.00mm, Capacitor_THT:C_Rect_L7.0mm_W2.5mm_P5.00mm, F.Cu at (54.0, 216.5)
Routing:
- net GND: track 0.00 -> 77.4 mm
- net OPAMP6: track 0.00 -> 55.8 mm
- net VCC: track 0.00 -> 50.6 mm
- net OPAMP1: track 0.00 -> 41.4 mm
- net OPAMP5: track 0.00 -> 24.8 mm
- net MICO: track 0.00 -> 17.9 mm
- net Poto1: track 0.00 -> 17.0 mm
- net OPAMP3: track 0.00 -> 14.0 mm
- net vmic: track 0.00 -> 11.6 mm
- net PATH1: track 0.00 -> 9.43 mm

Commit message: hello
Parts:
- added 74HC02: NOR, Package_SO:SOIC-14_3.9x8.7mm_P1.27mm, F.Cu at (111.2, 218.0)
- added 74HC08: AND, Package_SO:SOIC-14_3.9x8.7mm_P1.27mm, F.Cu at (99.2, 218.0)
- added 74HC14: NOT, Package_SO:SOIC-14_3.9x8.7mm_P1.27mm, F.Cu at (123.8, 218.0)
- added C5: ___uF, Capacitor_SMD:C_0805_2012Metric_Pad1.18x1.45mm_HandSolder, F.Cu at (107.0, 223.8)
- added C6: ___uF, Capacitor_SMD:C_0805_2012Metric_Pad1.18x1.45mm_HandSolder, F.Cu at (106.2, 210.5)
- added C7: ___uF, Capacitor_SMD:C_0805_2012Metric_Pad1.18x1.45mm_HandSolder, F.Cu at (118.8, 226.8)
- added C8: ___uF, Capacitor_SMD:C_0805_2012Metric_Pad1.18x1.45mm_HandSolder, F.Cu at (112.0, 211.8)
- added C9: ___uF, Capacitor_SMD:C_0805_2012Metric_Pad1.18x1.45mm_HandSolder, F.Cu at (118.8, 210.5)
- added Potentiometer: Potentiometer_Vishay_T73YP_Vertical, Potentiometer_THT:Potentiometer_Vishay_T73YP_Vertical, F.Cu at (115.5, 230.4)
- added Potentiometer: Potentiometer_Vishay_T73YP_Vertical, Potentiometer_THT:Potentiometer_Vishay_T73YP_Vertical, F.Cu at (128.8, 208.9)
- added Potentiometer: Potentiometer_Vishay_T73YP_Vertical, Potentiometer_THT:Potentiometer_Vishay_T73YP_Vertical, F.Cu at (129.0, 226.2)
- added Potentiometer: Potentiometer_Vishay_T73YP_Vertical, Potentiometer_THT:Potentiometer_Vishay_T73YP_Vertical, F.Cu at (115.5, 206.4)
- added R9: ___Ohm, Resistor_SMD:R_0805_2012Metric_Pad1.20x1.40mm_HandSolder, F.Cu at (102.5, 212.0)
Connections:
- Potentiometer pad 3: (no net) -> CUSTOM_Potentiometer-3_37
Routing:
- net GND: track 77.4 -> 3.65 mm
- net CUSTOM_74HC08-12_11: track 0.00 -> 29.0 mm
- net CUSTOM_74HC08-13_12: track 0.00 -> 23.6 mm
- net CUSTOM_74HC02-5_46: track 0.00 -> 23.4 mm
- net CUSTOM_74HC02-9_48: track 0.00 -> 20.4 mm, vias 0 -> 1
- net AND_8: track 0.00 -> 13.6 mm
- net CUSTOM_Potentiometer-3_20: track 0.00 -> 12.7 mm
- net output_c: track 0.00 -> 11.9 mm
- net CUSTOM_74HC08-3_5: track 0.00 -> 11.4 mm
- net CUSTOM_C8-2_55: track 0.00 -> 11.3 mm
- net COUT: track 0.00 -> 9.42 mm
- net vmic: track 11.6 -> 20.8 mm
- net AND_OUT: track 0.00 -> 5.95 mm
- net CUSTOM_74HC02-4_45: track 0.00 -> 3.89 mm
- net CUSTOM_74HC14-4_28: track 0.00 -> 1.27 mm
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- added copper zone on B.Cu, net GND
